Commit message: .

File: robots/aarya/exp10-robot/urdf/macros.xacro (robot description, xacro)
@@ -31,6 +31,4 @@
             <child link="${child}"/>
             <axis xyz="0 1 0"/>
-            <limit effort="1000" velocity="1000"/>
-            <joint_properties damping="1.0" friction="1.0"/>
         </joint>
     </xacro:macro>

File: robots/aarya/exp10-robot/urdf/materials.xacro (robot description, xacro)
@@ -1,20 +1,20 @@
 <?xml version="1.0"?>
-<robot name="exp10-robot" xmlns:xacro="http://www.ros.org/wiki/xacro">
-  <gazebo reference="left_back">
+<robot name="killer_robot" xmlns:xacro="http://www.ros.org/wiki/xacro">
+  <gazebo reference="back_left">
     <material>
       Gazebo/Blue
     </material>
   </gazebo>
-  <gazebo reference="right_back">
+  <gazebo reference="back_right">
     <material>
       Gazebo/Red
     </material>
   </gazebo>
-  <gazebo reference="right_front">
+  <gazebo reference="front_right">
     <material>
       Gazebo/Gold
     </material>
   </gazebo>
-<gazebo reference="left_front">
+<gazebo reference="front_left">
     <material>
       Gazebo/GoldGlow
@@ -34,9 +34,14 @@
       <leftRearJoint>back_left_joint</leftRearJoint>
       <rightRearJoint>back_right_joint</rightRearJoint>
-      <wheelSeparation>0.7</wheelSeparation>
+      <wheelSeparation>0.75</wheelSeparation>
       <wheelDiameter>${0.2*2}</wheelDiameter>
-      <robotBaseFrame>base_link</robotBaseFrame>
+      <robotBaseFrame>chassis</robotBaseFrame>
       <torque>20</torque>
-      <topicName>cmd_vel</topicName>
+      <commandTopic>cmd_vel</commandTopic>
+      <odometryTopic>odom</odometryTopic>
+      <odometryFrame>odom</odometryFrame>
+      <covariance_x>0.0001</covariance_x>
+      <covariance_y>0.0001</covariance_y>
+      <covariance_yaw>0.01</covariance_yaw>
       <broadcastTF>false</broadcastTF>
     </plugin>

File: robots/aarya/exp10-robot/urdf/model.xacro (robot description, xacro)
@@ -2,5 +2,4 @@
 <robot name="killer_robot" xmlns:xacro = "https://www.ros.org/wiki/xacro">
     <link name="chassis">
-        <pose>0 0 0.25 0 0 0</pose>
         <inertial>
             <origin xyz="0 0 0.25" rpy="0 0 0"/>
@@ -24,13 +23,13 @@
         </visual>
     </link>
+    <xacro:include filename="$(find exp10-robot)/urdf/macros.xacro"/>
+    <xacro:wheel_link link_name="front_right"/>
+    <xacro:wheel_link link_name="front_left"/>
+    <xacro:wheel_link link_name="back_right"/>
+    <xacro:wheel_link link_name="back_left"/>
+    <xacro:joint_link joint_name="front_right_joint" child="front_right" origin_xyz="1 0.375 0"/>
+    <xacro:joint_link joint_name="front_left_joint"  child="front_left"  origin_xyz="1 -0.375 0"/>
+    <xacro:joint_link joint_name="back_left_joint"   child="back_left"   origin_xyz="-1 0.375 0"/>
+    <xacro:joint_link joint_name="back_right_joint"  child="back_right"  origin_xyz="-1 -0.375 0"/>
     <xacro:include filename='$(find exp10-robot)/urdf/materials.xacro'/>
-    <xacro:include filename="$(find exp10-robot)/urdf/macros.xacro"/>
-    <xacro:wheel_link link_name="right_front"/>
-    <xacro:wheel_link link_name= "left_front"/>
-    <xacro:wheel_link link_name="right_back"/>
-    <xacro:wheel_link link_name="left_back"/>
-    <xacro:joint_link joint_name="right_front_joint" child="right_front" origin_xyz="1 0.375 0"/>
-    <xacro:joint_link joint_name="left_front_joint" child="left_front" origin_xyz="1 -0.375 0"/>
-    <xacro:joint_link joint_name="right_back_joint" child="right_back" origin_xyz="-1 0.375 0"/>
-    <xacro:joint_link joint_name="left_back_joint" child="left_back" origin_xyz="-1 -0.375 0"/>
 </robot>

File: robots/praveen/Robotics_project/Foxhead_012/urdf/materials.xacro (robot description, xacro)
@@ -8,18 +8,23 @@
     </gazebo>
     <gazebo>
-        <plugin filename="libgazebo_ros_robot_drive.so" name="4_wheeled_robot_controller">
-            <legacyMode>false</legacyMode>
-            <alwaysOn>true</alwaysOn>
-            <updateRate>20</updateRate>
-            <leftJoint>front_left_joint</leftJoint>
-            <rightJoint>front_right_joint</rightJoint>
-            <wheelSeparation>0.3</wheelSeparation>
-            <wheelDiameter>0.2</wheelDiameter>
-            <torque>0.1</torque>
-            <commandTopic>cmd_vel</commandTopic>
-            <odometryTopic>odom</odometryTopic>
-            <odometryFrame>odom</odometryFrame>
-            <robotBaseFrame>link_chassis</robotBaseFrame>
-        </plugin>
+      <plugin name="skid_steer_drive_controller" filename="libgazebo_ros_skid_steer_drive.so">
+        <updateRate>100.0</updateRate>
+        <robotNamespace>/</robotNamespace>
+        <leftFrontJoint>front_left_joint</leftFrontJoint>
+        <rightFrontJoint>front_right_joint</rightFrontJoint>
+        <leftRearJoint>rear_left_joint</leftRearJoint>
+        <rightRearJoint>rear_right_joint</rightRearJoint>
+        <wheelSeparation>0.3</wheelSeparation>
+        <wheelDiameter>0.2</wheelDiameter>
+        <robotBaseFrame>chassis</robotBaseFrame>
+        <torque>20</torque>
+        <commandTopic>cmd_vel</commandTopic>
+        <odometryTopic>odom</odometryTopic>
+        <odometryFrame>odom</odometryFrame>
+        <covariance_x>0.0001</covariance_x>
+        <covariance_y>0.0001</covariance_y>
+        <covariance_yaw>0.01</covariance_yaw>
+        <broadcastTF>false</broadcastTF>
+      </plugin>
     </gazebo>
 </robot>

File: robots/praveen/Robotics_project/Foxhead_012/urdf/model.xacro (robot description, xacro)
@@ -2,8 +2,7 @@
 <robot name="test_1" xmlns:xacro = "https://www.ros.org/wiki/xacro">
     <link name="chassis">
-        <pose>0 0 0.25 0 0 0</pose>
         <inertial>
             <origin xyz="0 0 0.25" rpy="0 0 0"/>
-            <mass value="5"/>
+            <mass value="50"/>
             <inertia ixx="0.046875" ixy="0" ixz="0" iyy="0.11354" iyz="0" izz="0.14167"/>
         </inertial>

File: robots/vidyut/robolab_mini_project/urdf/four_wheel_bot.xacro (robot description, xacro)
@@ -6,10 +6,9 @@
 <xacro:include filename="$(find robolab_mini_project)/urdf/materials.xacro" />
 <xacro:include filename="$(find robolab_mini_project)/urdf/macros.xacro" />
+<xacro:include filename="$(find robolab_mini_project)/urdf/four_wheel_bot.gazebo"/>
   <link name="base_link">
   <pose>0 0 3 0 0 0</pose>
     <visual>
-      <material name="orange">
-      	<color rgba="1 0.6 0 1"/>
-      </material>
+      <material name="orange"/>
       <origin xyz="0 0 0" rpy="0 0 0" />
       <geometry>

File: robots/vidyut/robolab_mini_project/urdf/macros.xacro (robot description, xacro)
@@ -1,4 +1,5 @@
 <?xml version="1.0"?>
 <robot name="four_wheel_bot" xmlns:xacro = "https://www.ros.org/wiki/xacro">
+<xacro:property name="wheel_radius" value="0.2"/>
     <xacro:macro name='wheel_link' params='link_name'>
         <link name="${link_name}">
@@ -17,9 +18,7 @@
                 <origin xyz="0 0 0" rpy="0 1.57 1.57"/>
                 <geometry>
-                    <cylinder radius="0.2" length="0.1"/>
+                    <cylinder radius="${wheel_radius}" length="0.1"/>
                 </geometry>
-                <material name="black">
-                  <color rgba="0.05 0.05 0.05 1"/>
-                </material>
+                <material name="black"/>
             </visual>
         </link>

File: robots/yash/yobot/urdf/yobot.xacro (robot description, xacro)
@@ -1,6 +1,4 @@
 <?xml version='1.0'?>
 <robot name="skid_steer_bot" xmlns:xacro="http://www.ros.org/wiki/xacro">
-  <xacro:property name="pi" value="3.1415926535897931"/>
-  <xacro:property name="DEG_TO_RAD" value="${PI/180.0}" />
   <xacro:property name="wheel_radius" value="0.2"/>
   <xacro:property name="wheel_thickness" value="0.2" />
