Commit message: .

File: robots/praveen/Robotics_project/Foxhead_012/urdf/materials.xacro (robot description, xacro)
@@ -15,8 +15,8 @@
         <leftRearJoint>rear_left_joint</leftRearJoint>
         <rightRearJoint>rear_right_joint</rightRearJoint>
-        <wheelSeparation>0.3</wheelSeparation>
+        <wheelSeparation>0.35</wheelSeparation>
         <wheelDiameter>0.2</wheelDiameter>
         <robotBaseFrame>chassis</robotBaseFrame>
-        <torque>20</torque>
+        <torque>0.55</torque>
         <commandTopic>cmd_vel</commandTopic>
         <odometryTopic>odom</odometryTopic>

File: robots/praveen/Robotics_project/Foxhead_012/urdf/model.xacro (robot description, xacro)
@@ -3,6 +3,5 @@
     <link name="chassis">
         <inertial>
-            <origin xyz="0 0 0.25" rpy="0 0 0"/>
-            <mass value="50"/>
+            <mass value="5"/>
             <inertia ixx="0.046875" ixy="0" ixz="0" iyy="0.11354" iyz="0" izz="0.14167"/>
         </inertial>
