Commit message: .

File: robots/pranav/ohno/urdf/robo.xacro (robot description, xacro)
@@ -3,9 +3,9 @@
   <xacro:property name="wheel_radius" value="0.2"/>
   <xacro:property name="wheel_thickness" value="0.1" />
-  <xacro:property name="wheel_mass" value="0.2" />
+  <xacro:property name="wheel_mass" value="0.1" />
   <xacro:property name="chassis_length" value="1" />
   <xacro:property name="chassis_breadth" value="0.5" />
   <xacro:property name="chassis_height" value="0.25" />
-  <xacro:property name="chassis_mass" value="5" />
+  <xacro:property name="chassis_mass" value="0.5" />
   <xacro:include filename="$(find ohno)/urdf/materials.xacro"/>
   <xacro:include filename="$(find ohno)/urdf/wheel.xacro"/>
@@ -13,5 +13,4 @@
   <!-- Base Link -->
   <link name="base_link">
-    <pose>0 0 3 0 0 0</pose>
     <visual>
       <material name="white"/>
@@ -33,7 +32,7 @@
     </inertial>
   </link>
-  <xacro:define_wheel name_a="front_right" name_b="front_right_joint" rad="${wheel_radius}" thicc="${wheel_thickness}" origin_xyz="0.4 -0.3 0.05"/>
-  <xacro:define_wheel name_a="front_left" name_b="front_left_joint" rad="${wheel_radius}" thicc="${wheel_thickness}" origin_xyz="0.4 0.3 0.05"/>
-  <xacro:define_wheel name_a="back_right" name_b="back_right_joint" rad="${wheel_radius}" thicc="${wheel_thickness}" origin_xyz="-0.4 -0.3 0.05"/>
-  <xacro:define_wheel name_a="back_left" name_b="back_left_joint" rad="${wheel_radius}" thicc="${wheel_thickness}" origin_xyz="-0.4 0.3 0.05"/>
+  <xacro:define_wheel name_a="front_right" name_b="front_right_joint" rad="${wheel_radius}" thicc="${wheel_thickness}" origin_xyz="0.4 -0.3 0"/>
+  <xacro:define_wheel name_a="front_left" name_b="front_left_joint" rad="${wheel_radius}" thicc="${wheel_thickness}" origin_xyz="0.4 0.3 0"/>
+  <xacro:define_wheel name_a="back_right" name_b="back_right_joint" rad="${wheel_radius}" thicc="${wheel_thickness}" origin_xyz="-0.4 -0.3 0"/>
+  <xacro:define_wheel name_a="back_left" name_b="back_left_joint" rad="${wheel_radius}" thicc="${wheel_thickness}" origin_xyz="-0.4 0.3 0"/>
 </robot>

File: robots/pranav/ohno/urdf/wheel.xacro (robot description, xacro)
@@ -6,5 +6,5 @@
         <link name="${name_a}">
             <inertial>
-                <mass value="0.5"/>
+                <mass value="0.05"/>
                 <inertia ixx="0.01" ixy="0" ixz="0" iyy="0.005" iyz="0" izz="0.005"/>
             </inertial>

File: robots/praveen/Robotics_project/Foxhead_012/urdf/model.xacro (robot description, xacro)
@@ -3,5 +3,5 @@
     <link name="chassis">
         <inertial>
-            <mass value="5"/>
+            <mass value="0.5"/>
             <inertia ixx="0.046875" ixy="0" ixz="0" iyy="0.11354" iyz="0" izz="0.14167"/>
         </inertial>
